File: board_designs/477breakout.sch (EAGLE design)
At the start: 18 parts, among them IC1 PIC24FJ128GA006, J1 RJ11-6PTH, J2 5.5x2.1mm Barrel, U2 3.3V/150mA, U3 5V

Commit message: Updated board designs
Parts:
- added C8, C9: 1 uF, rcl:C-USC0402
- added D1, D2, D3: 1N4004, diode:1N4004
- added JP10: M01PTH, SparkFun:M01PTH
- added JP5: (no value), SparkFun:M05
- added JP6: GND, SparkFun:M01PTH
- added JP7: 12V, SparkFun:M01PTH
- added JP8, JP9: (no value), SparkFun:M04PTH
- added Q1: TIP120, transistor-power:TIP120
- added R2: 1K, rcl:R-US_0204/7
- added U1: TXB0104, SparkFun-IC-Comms:TXB0104PWRSOIC14
- added U4: V_REG_MIC5205RT9069, SparkFun-IC-Power:V_REG_MIC5205RT9069
- C6, C7: value (none) -> 2.2 uF
Connections:
- new net 12V: C9.1, D2.A, Q1.C, U4.OUT
- new net N$10: JP9.1, U1.B4
- new net N$11: D1.A, D3.A, J2.PWR
- new net N$12: Q1.B, R2.2
- new net N$14: D2.C, JP7.1
- new net N$15: JP10.1, R2.1
- new net N$16: C8.1, D3.C, U4.EN, U4.IN
- new net N$3: JP8.4, U1.A1
- new net N$4: JP8.3, U1.A2
- new net N$5: JP8.2, U1.A3
- new net N$6: JP8.1, U1.A4
- new net N$7: JP9.4, U1.B1
- new net N$8: JP9.3, U1.B2
- new net N$9: JP9.2, U1.B3
- net 5V: now also JP5.1, JP5.2, JP5.3, JP5.4, JP5.5, U1.VCCB
- net GND: now also C8.2, C9.2, JP6.1, Q1.E, U1.GND, U4.GND
- net N$2: now also D1.C; no longer J2.PWR
- net VCC: now also U1.OE, U1.VCCA
Other:
- moved on the sheet: J1, J2
